Commit message: added compute_place_orientation and pick and place objectives plus new environment xacros

File: src/picknik_009_ur5e_config/description/environment_shelving_test.xacro (robot description, xacro)
@@ -7,6 +7,4 @@
     />
     <!-- Workcell (80/20 aluminum extrusion frame) -->
-    <!-- robot_mount in the Locus config is at xyz="0.28 -0.026 -0.2" rpy="0 0 pi/2" from workcell.
-         Since our robot is at world origin, we place the workcell at the inverse transform. -->
     <link name="workcell">
       <visual>
@@ -31,5 +29,5 @@
       <origin xyz="0.026 0.28 0.2" rpy="0 0 ${-pi/2}" />
     </joint>
-    <!-- Tote dimensions (matching Locus config) -->
+    <!-- Tote dimensions -->
     <xacro:property name="tote_x" value="${24 * 0.0254}" />
     <xacro:property name="tote_y" value="${15 * 0.0254}" />
@@ -37,5 +35,5 @@
     <xacro:property name="tote_wall" value="0.025" />
     <xacro:property name="tote_bottom" value="0.005" />
-    <!-- Left tote (positions relative to workcell frame, same as Locus config) -->
+    <!-- Left tote with lid — modeled as a solid box for collision avoidance -->
     <link name="left_tote_origin"/>
     <joint name="left_tote_origin_joint" type="fixed">
@@ -44,36 +42,27 @@
       <origin xyz="0.008 -0.055 -0.2189" rpy="0 0 ${pi}"/>
     </joint>
-    <xacro:generic_tote
-      parent="left_tote_origin"
-      prefix="left_"
-      x_length="${tote_x}"
-      y_length="${tote_y}"
-      z_length="${tote_z}"
-      side_wall_thickness="${tote_wall}"
-      bottom_thickness="${tote_bottom}"/>
-    <!-- Left tote lid (collision-only box on top of the left tote) -->
-    <link name="left_tote_lid">
+    <link name="left_tote_link">
       <visual>
         <geometry>
-          <box size="${tote_x} ${tote_y} ${tote_bottom}"/>
+          <box size="${tote_x} ${tote_y} ${tote_z}"/>
         </geometry>
-        <origin xyz="${tote_x/2} ${tote_y/2} 0"/>
-        <material name="tote_color">
-          <color rgba="0.5 0.5 0.5 0.5"/>
+        <origin xyz="${tote_x/2} ${tote_y/2} ${tote_z/2}"/>
+        <material name="tote_lid_color">
+          <color rgba="0.4 0.4 0.6 0.6"/>
         </material>
       </visual>
       <collision>
         <geometry>
-          <box size="${tote_x} ${tote_y} ${tote_bottom}"/>
+          <box size="${tote_x} ${tote_y} ${tote_z}"/>
         </geometry>
-        <origin xyz="${tote_x/2} ${tote_y/2} 0"/>
+        <origin xyz="${tote_x/2} ${tote_y/2} ${tote_z/2}"/>
       </collision>
     </link>
-    <joint name="left_tote_lid_joint" type="fixed">
+    <joint name="left_tote_joint" type="fixed">
       <parent link="left_tote_origin"/>
-      <child link="left_tote_lid"/>
-      <origin xyz="0 0 ${tote_z}" rpy="0 0 0"/>
+      <child link="left_tote_link"/>
+      <origin xyz="0 0 0" rpy="0 0 0"/>
     </joint>
-    <!-- Right tote -->
+    <!-- Right tote (keep as-is) -->
     <link name="right_tote_origin"/>
     <joint name="right_tote_origin_joint" type="fixed">
@@ -90,5 +79,5 @@
       side_wall_thickness="${tote_wall}"
       bottom_thickness="${tote_bottom}"/>
-    <!-- 80/20 camera mount bar (24" long, 1.75"x1.75", horizontal, 17.75" above workcell surface) -->
+    <!-- Camera mount bar -->
     <xacro:property name="bar_length" value="${24 * 0.0254}" />
     <xacro:property name="bar_cross" value="${1.75 * 0.0254}" />
@@ -113,5 +102,4 @@
       <parent link="${parent}" />
       <child link="camera_mount_bar" />
-      <!-- Center of bar: camera Y minus half bar length, at workcell surface + 17.75" -->
       <origin xyz="0.45 0.538 0.469" rpy="0 0 0" />
     </joint>

File: src/picknik_009_ur5e_config/description/grocery_item_collision.urdf (robot description, URDF)
Before this commit: robot grocery_item_collision, 1 links, 0 joints
Links:
- link grocery_item: geometry collision cylinder length=0.20 radius=0.04

File: src/picknik_009_ur5e_config/description/picknik_009_ur5e.urdf.xacro (robot description, xacro)
@@ -145,5 +145,6 @@
   </joint>
   <!-- Environment: table, walls, scene camera -->
-  <xacro:include filename="$(find picknik_009_ur5e_config)/description/environment.xacro"/>
+  <!-- Swap to environment_shelving_test.xacro to remove left tote for testing -->
+  <xacro:include filename="$(find picknik_009_ur5e_config)/description/environment_shelving_test.xacro"/>
   <xacro:environment parent="world"/>
 </robot>
