Commit message: current bin picker demo config

File: src/picknik_009_ur5e_config/description/environment.xacro (robot description, xacro)
@@ -4,5 +4,5 @@
     <!-- Import macros -->
     <xacro:include
-      filename="$(find picknik_accessories)/descriptions/sensors/realsense_d435.urdf.xacro"
+      filename="$(find picknik_accessories)/descriptions/sensors/extrinsic_calibrated_realsense.urdf.xacro"
     />
     <xacro:include
@@ -70,18 +70,38 @@
       side_wall_thickness="${tote_wall}"
       bottom_thickness="${tote_bottom}"/>
-    <!-- Scene camera (RealSense D435) -->
-    <link name="external_camera_link" />
-    <joint name="external_camera_joint" type="fixed">
+    <!-- 80/20 camera mount bar (24" long, 1.75"x1.75", horizontal, 17.75" above workcell surface) -->
+    <xacro:property name="bar_length" value="${24 * 0.0254}" />
+    <xacro:property name="bar_cross" value="${1.75 * 0.0254}" />
+    <link name="camera_mount_bar">
+      <visual>
+        <origin xyz="0 0 0" rpy="0 0 0" />
+        <geometry>
+          <box size="${bar_cross} ${bar_length} ${bar_cross}" />
+        </geometry>
+        <material name="aluminum_8020">
+          <color rgba="0.7 0.7 0.7 1" />
+        </material>
+      </visual>
+      <collision>
+        <origin xyz="0 0 0" rpy="0 0 0" />
+        <geometry>
+          <box size="${bar_cross} ${bar_length} ${bar_cross}" />
+        </geometry>
+      </collision>
+    </link>
+    <joint name="${parent}_to_camera_mount_bar" type="fixed">
       <parent link="${parent}" />
-      <child link="external_camera_link" />
-      <origin xyz="0.372 0.644 0.726" rpy="${-pi/2} 0 ${-pi/2}" />
+      <child link="camera_mount_bar" />
+      <!-- Center of bar: camera Y minus half bar length, at workcell surface + 17.75" -->
+      <origin xyz="0.45 0.538 0.469" rpy="0 0 0" />
     </joint>
-    <xacro:realsense_d435
-      parent="external_camera_link"
+    <!-- Scene camera (RealSense D415, pose loaded from calibration YAML) -->
+    <xacro:load_extrinsic_calibrated_realsense
       name="scene_camera"
-      visible="true"
-    >
-      <origin xyz="0 0 0" rpy="0 0 0" />
-    </xacro:realsense_d435>
+      parent="${parent}"
+      model="d415"
+      use_mesh="true"
+      extrinsic_calibration_parameter_file="$(find picknik_009_ur5e_config)/calibration/scene_camera_calibration.yaml"
+    />
   </xacro:macro>
 </robot>

File: src/picknik_009_ur5e_config/description/picknik_009_ur5e.urdf.xacro (robot description, xacro)
@@ -46,5 +46,5 @@
   <!-- EPick parameters -->
   <xacro:arg name="epick_extension_radius" default="0.005" />
-  <xacro:arg name="epick_extension_length" default="0.05" />
+  <xacro:arg name="epick_extension_length" default="0.08" />
   <xacro:arg name="epick_suction_cup_radius" default="0.012" />
   <xacro:arg name="epick_suction_cup_height" default="0.015" />

Commit message: added vacuum status checking

File: src/picknik_009_ur5e_config/description/environment.xacro (robot description, xacro)
@@ -3,7 +3,4 @@
   <xacro:macro name="environment" params="parent">
     <!-- Import macros -->
-    <xacro:include
-      filename="$(find picknik_accessories)/descriptions/sensors/extrinsic_calibrated_realsense.urdf.xacro"
-    />
     <xacro:include
       filename="$(find picknik_009_ur5e_config)/description/generic_tote.xacro"
@@ -45,5 +42,5 @@
       <parent link="workcell"/>
       <child link="left_tote_origin"/>
-      <origin xyz="0.008 -0.055 -0.21" rpy="0 0 ${pi}"/>
+      <origin xyz="0.008 -0.055 -0.2189" rpy="0 0 ${pi}"/>
     </joint>
     <xacro:generic_tote
@@ -60,5 +57,5 @@
       <parent link="workcell"/>
       <child link="right_tote_origin"/>
-      <origin xyz="0.008 0.4 -0.21" rpy="0 0 ${pi}"/>
+      <origin xyz="0.008 0.4 -0.2189" rpy="0 0 ${pi}"/>
     </joint>
     <xacro:generic_tote
@@ -96,12 +93,4 @@
       <origin xyz="0.45 0.538 0.469" rpy="0 0 0" />
     </joint>
-    <!-- Scene camera (RealSense D415, pose loaded from calibration YAML) -->
-    <xacro:load_extrinsic_calibrated_realsense
-      name="scene_camera"
-      parent="${parent}"
-      model="d415"
-      use_mesh="true"
-      extrinsic_calibration_parameter_file="$(find picknik_009_ur5e_config)/calibration/scene_camera_calibration.yaml"
-    />
   </xacro:macro>
 </robot>

File: src/picknik_009_ur5e_config/description/picknik_009_ur5e.urdf.xacro (robot description, xacro)
@@ -46,5 +46,5 @@
   <!-- EPick parameters -->
   <xacro:arg name="epick_extension_radius" default="0.005" />
-  <xacro:arg name="epick_extension_length" default="0.08" />
+  <xacro:arg name="epick_extension_length" default="0.088" />
   <xacro:arg name="epick_suction_cup_radius" default="0.012" />
   <xacro:arg name="epick_suction_cup_height" default="0.015" />

File: src/picknik_009_ur5e_config/description/picknik_009_ur5e_mujoco.urdf.xacro (robot description, xacro)
@@ -82,5 +82,5 @@
     parent="gripper_mount_link"
     extension_radius="0.005"
-    extension_length="0.05"
+    extension_length="0.088"
     suction_cup_radius="0.012"
     suction_cup_height="0.015"

Commit message: Add updated environment and config and custom behaviors

File: src/picknik_009_ur5e_config/description/environment.xacro (robot description, xacro)
@@ -1,9 +1,16 @@
 <?xml version="1.0" encoding="utf-8" ?>
 <robot xmlns:xacro="http://ros.org/wiki/xacro">
-  <xacro:macro name="environment" params="parent">
+  <xacro:macro name="environment" params="parent xyz:='0 0 0' rpy:='0 0 0'">
     <!-- Import macros -->
     <xacro:include
       filename="$(find picknik_009_ur5e_config)/description/generic_tote.xacro"
     />
+    <!-- Environment base link: move this to reposition the entire environment -->
+    <link name="environment_base" />
+    <joint name="${parent}_to_environment_base" type="fixed">
+      <parent link="${parent}" />
+      <child link="environment_base" />
+      <origin xyz="${xyz}" rpy="${rpy}" />
+    </joint>
     <!-- Workcell (80/20 aluminum extrusion frame) -->
     <!-- robot_mount in the Locus config is at xyz="0.28 -0.026 -0.2" rpy="0 0 pi/2" from workcell.
@@ -26,6 +33,6 @@
       </collision>
     </link>
-    <joint name="${parent}_to_workcell" type="fixed">
-      <parent link="${parent}" />
+    <joint name="environment_base_to_workcell" type="fixed">
+      <parent link="environment_base" />
       <child link="workcell" />
       <origin xyz="0.026 0.28 0.2" rpy="0 0 ${-pi/2}" />
@@ -38,5 +45,5 @@
     <xacro:property name="tote_bottom" value="0.005" />
     <!-- Left tote (positions relative to workcell frame, same as Locus config) -->
-    <link name="left_tote_origin"/>
+    <link name="left_tote_origin"/>0
     <joint name="left_tote_origin_joint" type="fixed">
       <parent link="workcell"/>
@@ -87,6 +94,6 @@
       </collision>
     </link>
-    <joint name="${parent}_to_camera_mount_bar" type="fixed">
-      <parent link="${parent}" />
+    <joint name="environment_base_to_camera_mount_bar" type="fixed">
+      <parent link="environment_base" />
       <child link="camera_mount_bar" />
       <!-- Center of bar: camera Y minus half bar length, at workcell surface + 17.75" -->

File: src/picknik_009_ur5e_config/description/picknik_009_ur5e.urdf.xacro (robot description, xacro)
@@ -146,4 +146,48 @@
   <!-- Environment: table, walls, scene camera -->
   <xacro:include filename="$(find picknik_009_ur5e_config)/description/environment.xacro"/>
-  <xacro:environment parent="world"/>
+  <xacro:environment parent="world" xyz="0.0 -1.41 0.115" rpy="0.0 0.0 0.0"/>
+  <link name="ur_stand">
+    <visual>
+      <origin xyz="0 0 0" rpy="0 0 0" />
+      <geometry>
+        <mesh filename="package://picknik_009_ur5e_config/description/ur_stand.stl" />
+      </geometry>
+      <material name="workcell_material">
+        <color rgba="0.792 0.820 0.933 1" />
+      </material>
+    </visual>
+    <collision>
+      <origin xyz="0 0 0" rpy="0 0 0" />
+      <geometry>
+        <mesh filename="package://picknik_009_ur5e_config/description/ur_stand.stl" />
+      </geometry>
+    </collision>
+  </link>
+  <joint name="world_to_ur_stand" type="fixed">
+    <parent link="world"/>
+    <child link="ur_stand"/>
+    <origin xyz="0.0 0.0 0" rpy="0.0 0.0 0.0"/>
+  </joint>
+  <link name="shelf">
+    <visual>
+      <origin xyz="0 0 0" rpy="0 0 0" />
+      <geometry>
+        <mesh filename="package://picknik_009_ur5e_config/description/shelf.stl" />
+      </geometry>
+      <material name="workcell_material">
+        <color rgba="0.792 0.820 0.933 1" />
+      </material>
+    </visual>
+    <collision>
+      <origin xyz="0 0 0" rpy="0 0 0" />
+      <geometry>
+        <mesh filename="package://picknik_009_ur5e_config/description/shelf.stl" />
+      </geometry>
+    </collision>
+  </link>
+  <joint name="world_to_shelf" type="fixed">
+    <parent link="world"/>
+    <child link="shelf"/>
+    <origin xyz="0.0 0.6096 -0.805" rpy="0.0 0.0 3.14159"/>
+  </joint>
 </robot>

Commit message: removed workcell from enviornment

File: src/picknik_009_ur5e_config/description/environment.xacro (robot description, xacro)
@@ -2,102 +2,5 @@
 <robot xmlns:xacro="http://ros.org/wiki/xacro">
   <xacro:macro name="environment" params="parent xyz:='0 0 0' rpy:='0 0 0'">
-    <!-- Import macros -->
-    <xacro:include
-      filename="$(find picknik_009_ur5e_config)/description/generic_tote.xacro"
-    />
-    <!-- Environment base link: move this to reposition the entire environment -->
-    <link name="environment_base" />
-    <joint name="${parent}_to_environment_base" type="fixed">
-      <parent link="${parent}" />
-      <child link="environment_base" />
-      <origin xyz="${xyz}" rpy="${rpy}" />
-    </joint>
-    <!-- Workcell (80/20 aluminum extrusion frame) -->
-    <!-- robot_mount in the Locus config is at xyz="0.28 -0.026 -0.2" rpy="0 0 pi/2" from workcell.
-         Since our robot is at world origin, we place the workcell at the inverse transform. -->
-    <link name="workcell">
-      <visual>
-        <origin xyz="0 0 0" rpy="0 0 0" />
-        <geometry>
-          <mesh filename="package://picknik_009_ur5e_config/meshes/workcell_no_totes.stl" />
-        </geometry>
-        <material name="workcell_material">
-          <color rgba="0.792 0.820 0.933 1" />
-        </material>
-      </visual>
-      <collision>
-        <origin xyz="0 0 0" rpy="0 0 0" />
-        <geometry>
-          <mesh filename="package://picknik_009_ur5e_config/meshes/workcell_no_totes.stl" />
-        </geometry>
-      </collision>
-    </link>
-    <joint name="environment_base_to_workcell" type="fixed">
-      <parent link="environment_base" />
-      <child link="workcell" />
-      <origin xyz="0.026 0.28 0.2" rpy="0 0 ${-pi/2}" />
-    </joint>
-    <!-- Tote dimensions (matching Locus config) -->
-    <xacro:property name="tote_x" value="${24 * 0.0254}" />
-    <xacro:property name="tote_y" value="${15 * 0.0254}" />
-    <xacro:property name="tote_z" value="${7.5 * 0.0254}" />
-    <xacro:property name="tote_wall" value="0.025" />
-    <xacro:property name="tote_bottom" value="0.005" />
-    <!-- Left tote (positions relative to workcell frame, same as Locus config) -->
-    <link name="left_tote_origin"/>
-    <joint name="left_tote_origin_joint" type="fixed">
-      <parent link="workcell"/>
-      <child link="left_tote_origin"/>
-      <origin xyz="0.008 -0.055 -0.2189" rpy="0 0 ${pi}"/>
-    </joint>
-    <xacro:generic_tote
-      parent="left_tote_origin"
-      prefix="left_"
-      x_length="${tote_x}"
-      y_length="${tote_y}"
-      z_length="${tote_z}"
-      side_wall_thickness="${tote_wall}"
-      bottom_thickness="${tote_bottom}"/>
-    <!-- Right tote -->
-    <link name="right_tote_origin"/>
-    <joint name="right_tote_origin_joint" type="fixed">
-      <parent link="workcell"/>
-      <child link="right_tote_origin"/>
-      <origin xyz="0.008 0.4 -0.2189" rpy="0 0 ${pi}"/>
-    </joint>
-    <xacro:generic_tote
-      parent="right_tote_origin"
-      prefix="right_"
-      x_length="${tote_x}"
-      y_length="${tote_y}"
-      z_length="${tote_z}"
-      side_wall_thickness="${tote_wall}"
-      bottom_thickness="${tote_bottom}"/>
-    <!-- 80/20 camera mount bar (24" long, 1.75"x1.75", horizontal, 17.75" above workcell surface) -->
-    <xacro:property name="bar_length" value="${24 * 0.0254}" />
-    <xacro:property name="bar_cross" value="${1.75 * 0.0254}" />
-    <link name="camera_mount_bar">
-      <visual>
-        <origin xyz="0 0 0" rpy="0 0 0" />
-        <geometry>
-          <box size="${bar_cross} ${bar_length} ${bar_cross}" />
-        </geometry>
-        <material name="aluminum_8020">
-          <color rgba="0.7 0.7 0.7 1" />
-        </material>
-      </visual>
-      <collision>
-        <origin xyz="0 0 0" rpy="0 0 0" />
-        <geometry>
-          <box size="${bar_cross} ${bar_length} ${bar_cross}" />
-        </geometry>
-      </collision>
-    </link>
-    <joint name="environment_base_to_camera_mount_bar" type="fixed">
-      <parent link="environment_base" />
-      <child link="camera_mount_bar" />
-      <!-- Center of bar: camera Y minus half bar length, at workcell surface + 17.75" -->
-      <origin xyz="0.45 0.538 0.469" rpy="0 0 0" />
-    </joint>
+    <!-- Environment removed for current setup -->
   </xacro:macro>
 </robot>

File: src/picknik_009_ur5e_config/description/picknik_009_ur5e.urdf.xacro (robot description, xacro)
@@ -144,50 +144,6 @@
     <origin xyz="0.0 0.0 0" rpy="0.0 0.0 0.0"/>
   </joint>
-  <!-- Environment: table, walls, scene camera -->
+  <!-- Environment removed for current setup -->
   <xacro:include filename="$(find picknik_009_ur5e_config)/description/environment.xacro"/>
-  <xacro:environment parent="world" xyz="0.0 -1.41 0.115" rpy="0.0 0.0 0.0"/>
-  <link name="ur_stand">
-    <visual>
-      <origin xyz="0 0 0" rpy="0 0 0" />
-      <geometry>
-        <mesh filename="package://picknik_009_ur5e_config/description/ur_stand.stl" />
-      </geometry>
-      <material name="workcell_material">
-        <color rgba="0.792 0.820 0.933 1" />
-      </material>
-    </visual>
-    <collision>
-      <origin xyz="0 0 0" rpy="0 0 0" />
-      <geometry>
-        <mesh filename="package://picknik_009_ur5e_config/description/ur_stand.stl" />
-      </geometry>
-    </collision>
-  </link>
-  <joint name="world_to_ur_stand" type="fixed">
-    <parent link="world"/>
-    <child link="ur_stand"/>
-    <origin xyz="0.0 0.0 0" rpy="0.0 0.0 0.0"/>
-  </joint>
-  <link name="shelf">
-    <visual>
-      <origin xyz="0 0 0" rpy="0 0 0" />
-      <geometry>
-        <mesh filename="package://picknik_009_ur5e_config/description/shelf.stl" />
-      </geometry>
-      <material name="workcell_material">
-        <color rgba="0.792 0.820 0.933 1" />
-      </material>
-    </visual>
-    <collision>
-      <origin xyz="0 0 0" rpy="0 0 0" />
-      <geometry>
-        <mesh filename="package://picknik_009_ur5e_config/description/shelf.stl" />
-      </geometry>
-    </collision>
-  </link>
-  <joint name="world_to_shelf" type="fixed">
-    <parent link="world"/>
-    <child link="shelf"/>
-    <origin xyz="0.0 0.6096 -0.805" rpy="0.0 0.0 3.14159"/>
-  </joint>
+  <xacro:environment parent="world"/>
 </robot>

Commit message: Update environment for table

File: src/picknik_009_ur5e_config/description/environment.xacro (robot description, xacro)
@@ -6,21 +6,15 @@
       filename="$(find picknik_009_ur5e_config)/description/generic_tote.xacro"
     />
-    <!-- Environment base link: move this to reposition the entire environment -->
-    <link name="environment_base" />
-    <joint name="${parent}_to_environment_base" type="fixed">
-      <parent link="${parent}" />
-      <child link="environment_base" />
-      <origin xyz="${xyz}" rpy="${rpy}" />
-    </joint>
-    <!-- Workcell (80/20 aluminum extrusion frame) -->
-    <!-- robot_mount in the Locus config is at xyz="0.28 -0.026 -0.2" rpy="0 0 pi/2" from workcell.
-         Since our robot is at world origin, we place the workcell at the inverse transform. -->
-    <link name="workcell">
+    <!-- Table (box geometry) -->
+    <xacro:property name="table_x" value="1.8288" />
+    <xacro:property name="table_y" value="0.46" />
+    <xacro:property name="table_z" value="0.74" />
+    <link name="table">
       <visual>
         <origin xyz="0 0 0" rpy="0 0 0" />
         <geometry>
-          <mesh filename="package://picknik_009_ur5e_config/meshes/workcell_no_totes.stl" />
+          <box size="${table_x} ${table_y} ${table_z}" />
         </geometry>
-        <material name="workcell_material">
+        <material name="table_material">
           <color rgba="0.792 0.820 0.933 1" />
         </material>
@@ -29,14 +23,14 @@
         <origin xyz="0 0 0" rpy="0 0 0" />
         <geometry>
-          <mesh filename="package://picknik_009_ur5e_config/meshes/workcell_no_totes.stl" />
+          <box size="${table_x} ${table_y} ${table_z}" />
         </geometry>
       </collision>
     </link>
-    <joint name="environment_base_to_workcell" type="fixed">
-      <parent link="environment_base" />
-      <child link="workcell" />
-      <origin xyz="0.026 0.28 0.2" rpy="0 0 ${-pi/2}" />
+    <joint name="${parent}_to_table" type="fixed">
+      <parent link="${parent}" />
+      <child link="table" />
+      <origin xyz="${xyz}" rpy="${rpy}" />
     </joint>
-    <!-- Tote dimensions (matching Locus config) -->
+    <!-- Tote dimensions -->
     <xacro:property name="tote_x" value="${24 * 0.0254}" />
     <xacro:property name="tote_y" value="${15 * 0.0254}" />
@@ -44,60 +38,18 @@
     <xacro:property name="tote_wall" value="0.025" />
     <xacro:property name="tote_bottom" value="0.005" />
-    <!-- Left tote (positions relative to workcell frame, same as Locus config) -->
-    <link name="left_tote_origin"/>0
-    <joint name="left_tote_origin_joint" type="fixed">
-      <parent link="workcell"/>
-      <child link="left_tote_origin"/>
-      <origin xyz="0.008 -0.055 -0.2189" rpy="0 0 ${pi}"/>
+    <link name="tote_origin" />
+    <joint name="table_to_tote_origin" type="fixed">
+      <parent link="table" />
+      <child link="tote_origin" />
+      <origin xyz="${-tote_x / 2} ${table_y / 2 - tote_y} ${table_z / 2}" rpy="0 0 0" />
     </joint>
     <xacro:generic_tote
-      parent="left_tote_origin"
-      prefix="left_"
+      parent="tote_origin"
+      prefix=""
       x_length="${tote_x}"
       y_length="${tote_y}"
       z_length="${tote_z}"
       side_wall_thickness="${tote_wall}"
-      bottom_thickness="${tote_bottom}"/>
-    <!-- Right tote -->
-    <link name="right_tote_origin"/>
-    <joint name="right_tote_origin_joint" type="fixed">
-      <parent link="workcell"/>
-      <child link="right_tote_origin"/>
-      <origin xyz="0.008 0.4 -0.2189" rpy="0 0 ${pi}"/>
-    </joint>
-    <xacro:generic_tote
-      parent="right_tote_origin"
-      prefix="right_"
-      x_length="${tote_x}"
-      y_length="${tote_y}"
-      z_length="${tote_z}"
-      side_wall_thickness="${tote_wall}"
-      bottom_thickness="${tote_bottom}"/>
-    <!-- 80/20 camera mount bar (24" long, 1.75"x1.75", horizontal, 17.75" above workcell surface) -->
-    <xacro:property name="bar_length" value="${24 * 0.0254}" />
-    <xacro:property name="bar_cross" value="${1.75 * 0.0254}" />
-    <link name="camera_mount_bar">
-      <visual>
-        <origin xyz="0 0 0" rpy="0 0 0" />
-        <geometry>
-          <box size="${bar_cross} ${bar_length} ${bar_cross}" />
-        </geometry>
-        <material name="aluminum_8020">
-          <color rgba="0.7 0.7 0.7 1" />
-        </material>
-      </visual>
-      <collision>
-        <origin xyz="0 0 0" rpy="0 0 0" />
-        <geometry>
-          <box size="${bar_cross} ${bar_length} ${bar_cross}" />
-        </geometry>
-      </collision>
-    </link>
-    <joint name="environment_base_to_camera_mount_bar" type="fixed">
-      <parent link="environment_base" />
-      <child link="camera_mount_bar" />
-      <!-- Center of bar: camera Y minus half bar length, at workcell surface + 17.75" -->
-      <origin xyz="0.45 0.538 0.469" rpy="0 0 0" />
-    </joint>
+      bottom_thickness="${tote_bottom}" />
   </xacro:macro>
 </robot>

File: src/picknik_009_ur5e_config/description/picknik_009_ur5e.urdf.xacro (robot description, xacro)
@@ -146,5 +146,5 @@
   <!-- Environment: table, walls, scene camera -->
   <xacro:include filename="$(find picknik_009_ur5e_config)/description/environment.xacro"/>
-  <xacro:environment parent="world" xyz="0.0 -1.41 0.115" rpy="0.0 0.0 0.0"/>
+  <xacro:environment parent="world" xyz="0.0 -0.78 -0.435" rpy="0.0 0.0 0.0"/>
   <link name="ur_stand">
     <visual>
@@ -189,5 +189,5 @@
     <parent link="world"/>
     <child link="shelf"/>
-    <origin xyz="0.0 0.6096 -0.805" rpy="0.0 0.0 3.14159"/>
+    <origin xyz="0.0 0.66 -0.805" rpy="0.0 0.0 3.14159"/>
   </joint>
 </robot>
