Commit message: increased path tolerance to 5 deg added calibration behavior

File: src/picknik_009_ur5e_config/description/environment.xacro (robot description, xacro)
@@ -42,5 +42,5 @@
       <parent link="table" />
       <child link="tote_origin" />
-      <origin xyz="${-tote_x / 2} ${table_y / 2 - tote_y} ${table_z / 2}" rpy="0 0 0" />
+      <origin xyz="${-tote_x / 2} ${table_y / 2 - tote_y - 0.04} ${table_z / 2}" rpy="0 0 0" />
     </joint>
     <xacro:generic_tote
@@ -52,4 +52,37 @@
       side_wall_thickness="${tote_wall}"
       bottom_thickness="${tote_bottom}" />
+    <!-- Scene camera pole: 28" tall, 1" radius cylinder, centered behind the bin -->
+    <xacro:property name="pole_height" value="${28 * 0.0254}" />
+    <xacro:property name="pole_radius" value="${1 * 0.0254}" />
+    <link name="scene_camera_pole">
+      <visual>
+        <origin xyz="0 0 0" rpy="0 0 0" />
+        <geometry>
+          <cylinder radius="${pole_radius}" length="${pole_height}" />
+        </geometry>
+        <material name="pole_material">
+          <color rgba="0.5 0.5 0.5 1" />
+        </material>
+      </visual>
+      <collision>
+        <origin xyz="0 0 0" rpy="0 0 0" />
+        <geometry>
+          <cylinder radius="${pole_radius}" length="${pole_height}" />
+        </geometry>
+      </collision>
+    </link>
+    <joint name="table_to_scene_camera_pole" type="fixed">
+      <parent link="table" />
+      <child link="scene_camera_pole" />
+      <!-- Centered on bin in X, at far edge of bin in Y, pole center above table top -->
+      <origin xyz="0 ${table_y / 2 - tote_y - 0.04} ${table_z / 2 + pole_height / 2}" rpy="0 0 0" />
+    </joint>
+    <!-- Mount point at pole top, shifted 3cm toward robot (+Y in table frame) -->
+    <link name="scene_camera_mount" />
+    <joint name="pole_to_scene_camera_mount" type="fixed">
+      <parent link="table" />
+      <child link="scene_camera_mount" />
+      <origin xyz="0 ${table_y / 2 - tote_y - 0.04 + 0.03} ${table_z / 2 + pole_height}" rpy="0 0 0" />
+    </joint>
   </xacro:macro>
 </robot>

File: src/picknik_009_ur5e_config/description/picknik_009_ur5e.urdf.xacro (robot description, xacro)
@@ -144,7 +144,15 @@
     <origin xyz="0.0 0.0 0" rpy="0.0 0.0 0.0"/>
   </joint>
-  <!-- Environment: table, walls, scene camera -->
+  <!-- Environment: table, tote, scene camera pole -->
   <xacro:include filename="$(find picknik_009_ur5e_config)/description/environment.xacro"/>
-  <xacro:environment parent="world" xyz="0.0 -0.78 -0.435" rpy="0.0 0.0 0.0"/>
+  <xacro:environment parent="world" xyz="0.0 -0.74 -0.435" rpy="0.0 0.0 0.0"/>
+  <!-- Scene camera (D415) on pole above bin, facing down at 75 degrees -->
+  <xacro:realsense_d415
+    parent="scene_camera_mount"
+    name="scene_camera"
+    use_mesh="true"
+  >
+    <origin xyz="0 0 0" rpy="${pi} ${75 * pi / 180} ${pi / 2}" />
+  </xacro:realsense_d415>
   <link name="ur_stand">
     <visual>
@@ -169,25 +177,5 @@
     <origin xyz="0.0 0.0 0" rpy="0.0 0.0 0.0"/>
   </joint>
-  <link name="shelf">
-    <visual>
-      <origin xyz="0 0 0" rpy="0 0 0" />
-      <geometry>
-        <mesh filename="package://picknik_009_ur5e_config/description/shelf.stl" />
-      </geometry>
-      <material name="workcell_material">
-        <color rgba="0.792 0.820 0.933 1" />
-      </material>
-    </visual>
-    <collision>
-      <origin xyz="0 0 0" rpy="0 0 0" />
-      <geometry>
-        <mesh filename="package://picknik_009_ur5e_config/description/shelf.stl" />
-      </geometry>
-    </collision>
-  </link>
-  <joint name="world_to_shelf" type="fixed">
-    <parent link="world"/>
-    <child link="shelf"/>
-    <origin xyz="0.0 0.66 -0.805" rpy="0.0 0.0 3.14159"/>
-  </joint>
+  <!-- Shelf is placed dynamically by the "Calibrate Qualcomm Setup" objective
+       using AprilTag-based calibration.  Do not add a static shelf here. -->
 </robot>

Commit message: added calibration, nathan edit to srdf and confidence sorting behaviors

File: src/picknik_009_ur5e_config/description/environment.xacro (robot description, xacro)
@@ -2,87 +2,7 @@
 <robot xmlns:xacro="http://ros.org/wiki/xacro">
   <xacro:macro name="environment" params="parent xyz:='0 0 0' rpy:='0 0 0'">
-    <!-- Import macros -->
-    <xacro:include
-      filename="$(find picknik_009_ur5e_config)/description/generic_tote.xacro"
-    />
-    <!-- Table (box geometry) -->
-    <xacro:property name="table_x" value="1.8288" />
-    <xacro:property name="table_y" value="0.46" />
-    <xacro:property name="table_z" value="0.74" />
-    <link name="table">
-      <visual>
-        <origin xyz="0 0 0" rpy="0 0 0" />
-        <geometry>
-          <box size="${table_x} ${table_y} ${table_z}" />
-        </geometry>
-        <material name="table_material">
-          <color rgba="0.792 0.820 0.933 1" />
-        </material>
-      </visual>
-      <collision>
-        <origin xyz="0 0 0" rpy="0 0 0" />
-        <geometry>
-          <box size="${table_x} ${table_y} ${table_z}" />
-        </geometry>
-      </collision>
-    </link>
-    <joint name="${parent}_to_table" type="fixed">
-      <parent link="${parent}" />
-      <child link="table" />
-      <origin xyz="${xyz}" rpy="${rpy}" />
-    </joint>
-    <!-- Tote dimensions -->
-    <xacro:property name="tote_x" value="${24 * 0.0254}" />
-    <xacro:property name="tote_y" value="${15 * 0.0254}" />
-    <xacro:property name="tote_z" value="${7.5 * 0.0254}" />
-    <xacro:property name="tote_wall" value="0.025" />
-    <xacro:property name="tote_bottom" value="0.005" />
-    <link name="tote_origin" />
-    <joint name="table_to_tote_origin" type="fixed">
-      <parent link="table" />
-      <child link="tote_origin" />
-      <origin xyz="${-tote_x / 2} ${table_y / 2 - tote_y - 0.04} ${table_z / 2}" rpy="0 0 0" />
-    </joint>
-    <xacro:generic_tote
-      parent="tote_origin"
-      prefix=""
-      x_length="${tote_x}"
-      y_length="${tote_y}"
-      z_length="${tote_z}"
-      side_wall_thickness="${tote_wall}"
-      bottom_thickness="${tote_bottom}" />
-    <!-- Scene camera pole: 28" tall, 1" radius cylinder, centered behind the bin -->
-    <xacro:property name="pole_height" value="${28 * 0.0254}" />
-    <xacro:property name="pole_radius" value="${1 * 0.0254}" />
-    <link name="scene_camera_pole">
-      <visual>
-        <origin xyz="0 0 0" rpy="0 0 0" />
-        <geometry>
-          <cylinder radius="${pole_radius}" length="${pole_height}" />
-        </geometry>
-        <material name="pole_material">
-          <color rgba="0.5 0.5 0.5 1" />
-        </material>
-      </visual>
-      <collision>
-        <origin xyz="0 0 0" rpy="0 0 0" />
-        <geometry>
-          <cylinder radius="${pole_radius}" length="${pole_height}" />
-        </geometry>
-      </collision>
-    </link>
-    <joint name="table_to_scene_camera_pole" type="fixed">
-      <parent link="table" />
-      <child link="scene_camera_pole" />
-      <!-- Centered on bin in X, at far edge of bin in Y, pole center above table top -->
-      <origin xyz="0 ${table_y / 2 - tote_y - 0.04} ${table_z / 2 + pole_height / 2}" rpy="0 0 0" />
-    </joint>
-    <!-- Mount point at pole top, shifted 3cm toward robot (+Y in table frame) -->
-    <link name="scene_camera_mount" />
-    <joint name="pole_to_scene_camera_mount" type="fixed">
-      <parent link="table" />
-      <child link="scene_camera_mount" />
-      <origin xyz="0 ${table_y / 2 - tote_y - 0.04 + 0.03} ${table_z / 2 + pole_height}" rpy="0 0 0" />
-    </joint>
+    <!-- All environment objects (table, bin, pole, camera) are now placed dynamically
+         by the "Calibrate Bin" and "Load Calibrated Scene" objectives.
+         Do not add static objects here. -->
   </xacro:macro>
 </robot>

File: src/picknik_009_ur5e_config/description/picknik_009_ur5e.urdf.xacro (robot description, xacro)
@@ -144,8 +144,17 @@
     <origin xyz="0.0 0.0 0" rpy="0.0 0.0 0.0"/>
   </joint>
-  <!-- Environment: table, tote, scene camera pole -->
+  <!-- Environment objects (table, bin, pole, camera) are placed dynamically
+       by the "Calibrate Bin" and "Load Calibrated Scene" objectives. -->
   <xacro:include filename="$(find picknik_009_ur5e_config)/description/environment.xacro"/>
-  <xacro:environment parent="world" xyz="0.0 -0.74 -0.435" rpy="0.0 0.0 0.0"/>
-  <!-- Scene camera (D415) on pole above bin, facing down at 75 degrees -->
+  <xacro:environment parent="world"/>
+  <!-- Scene camera (D415) at calibrated mount position above bin.
+       Position from calibration/camera_calibrated_pose.yaml.
+       Orientation: flipped (roll=pi), pitched 75 deg down, rotated 90 deg yaw. -->
+  <link name="scene_camera_mount" />
+  <joint name="world_to_scene_camera_mount" type="fixed">
+    <parent link="world" />
+    <child link="scene_camera_mount" />
+    <origin xyz="0.046 -0.984 0.563" rpy="0 0 0" />
+  </joint>
   <xacro:realsense_d415
     parent="scene_camera_mount"
@@ -153,5 +162,5 @@
     use_mesh="true"
   >
-    <origin xyz="0 0 0" rpy="${pi} ${75 * pi / 180} ${pi / 2}" />
+    <origin xyz="0 0 0" rpy="${pi} ${100 * pi / 180} ${-pi / 2}" />
   </xacro:realsense_d415>
   <link name="ur_stand">
