Commit message: mujoco sim works for teleop and camera

File: src/picknik_009_ur5e_config/description/picknik_009_ur5e.urdf.xacro (robot description, xacro)
@@ -52,4 +52,6 @@
   <!-- convert to property to use substitution in function -->
   <xacro:property name="initial_positions_file" default="$(arg initial_positions_file)"/>
+  <xacro:property name="use_fake_hardware_prop" value="$(arg use_fake_hardware)"/>
+  <xacro:property name="generate_ros2_control" value="${'false' if use_fake_hardware_prop else 'true'}" />
   <!-- create link fixed to the "world" -->
   <link name="world" />
@@ -91,4 +93,5 @@
           script_sender_port="$(arg script_sender_port)"
           trajectory_port="$(arg trajectory_port)"
+          generate_ros2_control_tag="${generate_ros2_control}"
   >
     <origin xyz="0 0 0" rpy="0 0 0" />
@@ -173,3 +176,7 @@
   <!-- Shelf is placed dynamically by the "Calibrate Qualcomm Setup" objective
        using AprilTag-based calibration.  Do not add a static shelf here. -->
+  <!-- Include MuJoCo ros2_control when using fake hardware (simulation) -->
+  <xacro:if value="$(arg use_fake_hardware)">
+    <xacro:include filename="$(find picknik_009_ur5e_config_sim)/urdf/ur_mujoco_ros2_control.xacro"/>
+  </xacro:if>
 </robot>

Commit message: mujoco sim works for teleop and camera

File: src/picknik_009_ur5e_config/description/picknik_009_ur5e.urdf.xacro (robot description, xacro)
@@ -52,4 +52,6 @@
   <!-- convert to property to use substitution in function -->
   <xacro:property name="initial_positions_file" default="$(arg initial_positions_file)"/>
+  <xacro:property name="use_fake_hardware_prop" value="$(arg use_fake_hardware)"/>
+  <xacro:property name="generate_ros2_control" value="${'false' if use_fake_hardware_prop else 'true'}" />
   <!-- create link fixed to the "world" -->
   <link name="world" />
@@ -91,4 +93,5 @@
           script_sender_port="$(arg script_sender_port)"
           trajectory_port="$(arg trajectory_port)"
+          generate_ros2_control_tag="${generate_ros2_control}"
   >
     <origin xyz="0 0 0" rpy="0 0 0" />
@@ -147,3 +150,7 @@
   <xacro:include filename="$(find picknik_009_ur5e_config)/description/environment.xacro"/>
   <xacro:environment parent="world"/>
+  <!-- Include MuJoCo ros2_control when using fake hardware (simulation) -->
+  <xacro:if value="$(arg use_fake_hardware)">
+    <xacro:include filename="$(find picknik_009_ur5e_config_sim)/urdf/ur_mujoco_ros2_control.xacro"/>
+  </xacro:if>
 </robot>

Commit message: adding in calibration yamls, meshes, and behaviors ... currently can shelve

File: src/picknik_009_ur5e_config/description/picknik_009_ur5e.urdf.xacro (robot description, xacro)
@@ -46,5 +46,5 @@
   <!-- EPick parameters -->
   <xacro:arg name="epick_extension_radius" default="0.005" />
-  <xacro:arg name="epick_extension_length" default="0.088" />
+  <xacro:arg name="epick_extension_length" default="0.1" />
   <xacro:arg name="epick_suction_cup_radius" default="0.012" />
   <xacro:arg name="epick_suction_cup_height" default="0.015" />
@@ -148,20 +148,5 @@
   <xacro:include filename="$(find picknik_009_ur5e_config)/description/environment.xacro"/>
   <xacro:environment parent="world"/>
-  <!-- Scene camera (D415) at calibrated mount position above bin.
-       Position from calibration/camera_calibrated_pose.yaml.
-       Orientation: flipped (roll=pi), pitched 75 deg down, rotated 90 deg yaw. -->
-  <link name="scene_camera_mount" />
-  <joint name="world_to_scene_camera_mount" type="fixed">
-    <parent link="world" />
-    <child link="scene_camera_mount" />
-    <origin xyz="0.046 -0.984 0.563" rpy="0 0 0" />
-  </joint>
-  <xacro:realsense_d415
-    parent="scene_camera_mount"
-    name="scene_camera"
-    use_mesh="true"
-  >
-    <origin xyz="0 0 0" rpy="${pi} ${100 * pi / 180} ${-pi / 2}" />
-  </xacro:realsense_d415>
+  <!-- Scene camera is placed dynamically by calibration objectives. -->
   <link name="ur_stand">
     <visual>
