Commit message: update robot_description.urdf to use collision stls and add inertial properties for vacuum link

File: src/picknik_009_ur5e_config_sim/mjcf/assets/robot_description.urdf (robot description, URDF)
Before this commit: robot ur5e, 43 links, 42 joints
Links:
- link base_link_inertia: geometry collision mesh filename=package://ur_description/meshes/ur5e/collision/base.stl; visual mesh filename=package://ur_description/meshes/ur5e/collision/base.stl
- link epick_vacuum_state: mass None -> 0.01
- link forearm_link: geometry collision mesh filename=package://ur_description/meshes/ur5e/collision/forearm.stl; visual mesh filename=package://ur_description/meshes/ur5e/collision/forearm.stl
- link shoulder_link: geometry collision mesh filename=package://ur_description/meshes/ur5e/collision/shoulder.stl; visual mesh filename=package://ur_description/meshes/ur5e/collision/shoulder.stl
- link upper_arm_link: geometry collision mesh filename=package://ur_description/meshes/ur5e/collision/upperarm.stl; visual mesh filename=package://ur_description/meshes/ur5e/collision/upperarm.stl
- link ur_to_robotiq_link: geometry collision mesh filename=package://robotiq_description/meshes/collision/2f_85/ur_to_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; visual mesh filename=package://robotiq_description/meshes/collision/2f_85/ur_to_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
- link wrist_1_link: geometry collision mesh filename=package://ur_description/meshes/ur5e/collision/wrist1.stl; visual mesh filename=package://ur_description/meshes/ur5e/collision/wrist1.stl
- link wrist_2_link: geometry collision mesh filename=package://ur_description/meshes/ur5e/collision/wrist2.stl; visual mesh filename=package://ur_description/meshes/ur5e/collision/wrist2.stl
- link wrist_3_link: geometry collision mesh filename=package://ur_description/meshes/ur5e/collision/wrist3.stl; visual mesh filename=package://ur_description/meshes/ur5e/collision/wrist3.stl
- link wrist_mounted_camera_link: geometry collision box size=0.02005 0.099 0.023; visual box size=0.02005 0.099 0.023

Commit message: update mujoco model to match real, apply pre-commit

File: src/picknik_009_ur5e_config_sim/mjcf/assets/robot_description.urdf (robot description, URDF)
Before this commit: robot ur5e, 43 links, 42 joints
Links:
- removed link camera_mount_bar
- removed link left_tote_link
- removed link left_tote_origin
- removed link right_tote_link
- removed link right_tote_origin
Joints:
- removed joint left_tote_joint
- removed joint left_tote_origin_joint
- removed joint right_tote_joint
- removed joint right_tote_origin_joint
- removed joint world_to_camera_mount_bar

File: src/picknik_009_ur5e_config_sim/urdf/ur_mujoco_ros2_control.xacro (robot description, xacro)
@@ -10,5 +10,5 @@
       <param name="tf_publish_rate">60</param>
       <param name="lidar_publish_rate">10</param>
-      <param name="mujoco_viewer">false</param>
+      <param name="mujoco_viewer">true</param>
     </hardware>
     <joint name="shoulder_pan_joint">
