Commit message: Remove obsolete URDF file for UR5e robot description to streamline the project structure and avoid confusion with autogenerated files.

File: src/ur_sim/description/picknik_ur.xacro (robot description, xacro)
@@ -67,11 +67,4 @@
     <origin xyz="0 0 0" rpy="0 0 0" />          <!-- position robot in the world -->
   </xacro:ur_robot>
-  <!-- ros2_control mock hardware -->
-  <!-- <xacro:include filename="$(find ur_description)/urdf/ros2_control_mock_hardware.xacro"/>
-  <xacro:ur_ros2_control
-    name="$(arg name)"
-    tf_prefix="$(arg tf_prefix)"
-    mock_sensor_commands="$(arg mock_sensor_commands)"
-  /> -->
   <!-- wrist camera adapter and camera-->
   <xacro:include
@@ -108,14 +101,352 @@
     rotation="0"
   />
-  <xacro:robotiq_gripper
-    name="RobotiqGripperHardwareInterface"
-    prefix="$(arg tf_prefix)"
-    parent="gripper_mount_link"
-    use_fake_hardware="$(arg use_fake_hardware)"
-    sim_ignition="false"
-    com_port="$(arg tool_device_name)"
-  >
-    <origin xyz="0 0 0" rpy="0 0 0" />
-  </xacro:robotiq_gripper>
+  <link name="robotiq_85_base_link">
+    <visual>
+      <geometry>
+        <mesh
+          filename="package://robotiq_description/meshes/visual/2f_85/robotiq_base.dae"
+        />
+      </geometry>
+    </visual>
+    <collision>
+      <geometry>
+        <mesh
+          filename="package://robotiq_description/meshes/collision/2f_85/robotiq_base.stl"
+        />
+      </geometry>
+    </collision>
+    <inertial>
+      <origin rpy="0 0 0" xyz="0.0 2.274e-05 0.03232288" />
+      <mass value="6.6320197e-01" />
+      <inertia
+        ixx="5.1617816e-04"
+        ixy="2.936e-8"
+        ixz="0.0"
+        iyy="5.8802208e-04"
+        iyz="-3.2296e-7"
+        izz="3.9462776e-04"
+      />
+    </inertial>
+  </link>
+  <link name="robotiq_85_left_knuckle_link">
+    <visual>
+      <geometry>
+        <mesh
+          filename="package://robotiq_description/meshes/visual/2f_85/left_knuckle.dae"
+        />
+      </geometry>
+    </visual>
+    <collision>
+      <geometry>
+        <mesh
+          filename="package://robotiq_description/meshes/collision/2f_85/left_knuckle.stl"
+        />
+      </geometry>
+    </collision>
+    <inertial>
+      <origin rpy="0 0 0" xyz="0.01213197 0.0002 -0.00058647" />
+      <mass value="1.384773208e-02" />
+      <inertia
+        ixx="3.5232e-7"
+        ixy="0.0"
+        ixz="1.1744e-7"
+        iyy="2.31944e-6"
+        iyz="0"
+        izz="2.23136e-6"
+      />
+    </inertial>
+  </link>
+  <link name="robotiq_85_right_knuckle_link">
+    <visual>
+      <geometry>
+        <mesh
+          filename="package://robotiq_description/meshes/visual/2f_85/right_knuckle.dae"
+        />
+      </geometry>
+    </visual>
+    <collision>
+      <geometry>
+        <mesh
+          filename="package://robotiq_description/meshes/collision/2f_85/right_knuckle.stl"
+        />
+      </geometry>
+    </collision>
+    <inertial>
+      <origin rpy="0 0 0" xyz="-0.01213197 0.0002 -0.00058647" />
+      <mass value="1.384773208e-02" />
+      <inertia
+        ixx="3.5232e-7"
+        ixy="0.0"
+        ixz="-1.1744e-7"
+        iyy="2.31944e-6"
+        iyz="0.0"
+        izz="2.23136e-6"
+      />
+    </inertial>
+  </link>
+  <link name="robotiq_85_left_finger_link">
+    <visual>
+      <geometry>
+        <mesh
+          filename="package://robotiq_description/meshes/visual/2f_85/left_finger.dae"
+        />
+      </geometry>
+    </visual>
+    <collision>
+      <geometry>
+        <mesh
+          filename="package://robotiq_description/meshes/collision/2f_85/left_finger.stl"
+        />
+      </geometry>
+    </collision>
+    <inertial>
+      <origin rpy="0 0 0" xyz="0.00346899 -0.00079447 0.01867121" />
+      <mass value="4.260376752e-02" />
+      <inertia
+        ixx="1.385792000000000e-05"
+        ixy="0.0"
+        ixz="-2.17264e-06"
+        iyy="1.183208e-05"
+        iyz="0.0"
+        izz="5.19672e-06"
+      />
+    </inertial>
+  </link>
+  <link name="robotiq_85_right_finger_link">
+    <visual>
+      <geometry>
+        <mesh
+          filename="package://robotiq_description/meshes/visual/2f_85/right_finger.dae"
+        />
+      </geometry>
+    </visual>
+    <collision>
+      <geometry>
+        <mesh
+          filename="package://robotiq_description/meshes/collision/2f_85/right_finger.stl"
+        />
+      </geometry>
+    </collision>
+    <inertial>
+      <origin rpy="0 0 0" xyz="-0.00346899 -5.53e-06 0.01867121" />
+      <mass value="4.260376752000000e-02" />
+      <inertia
+        ixx="1.385792e-05"
+        ixy="0.0"
+        ixz="2.17264e-06"
+        iyy="1.183208e-05"
+        iyz="0.0"
+        izz="5.19672e-06"
+      />
+    </inertial>
+  </link>
+  <link name="robotiq_85_left_inner_knuckle_link">
+    <visual>
+      <geometry>
+        <mesh
+          filename="package://robotiq_description/meshes/visual/2f_85/left_inner_knuckle.dae"
+        />
+      </geometry>
+    </visual>
+    <collision>
+      <geometry>
+        <mesh
+          filename="package://robotiq_description/meshes/collision/2f_85/left_inner_knuckle.stl"
+        />
+      </geometry>
+    </collision>
+    <inertial>
+      <origin rpy="0 0 0" xyz="0.01897699 0.00015001 0.02247101" />
+      <mass value="2.969376448e-02" />
+      <inertia
+        ixx="9.57136e-06"
+        ixy="0.0"
+        ixz="-3.93424e-06"
+        iyy="8.69056e-06"
+        iyz="0.0"
+        izz="8.19144e-06"
+      />
+    </inertial>
+  </link>
+  <link name="robotiq_85_right_inner_knuckle_link">
+    <visual>
+      <geometry>
+        <mesh
+          filename="package://robotiq_description/meshes/visual/2f_85/right_inner_knuckle.dae"
+        />
+      </geometry>
+    </visual>
+    <collision>
+      <geometry>
+        <mesh
+          filename="package://robotiq_description/meshes/collision/2f_85/right_inner_knuckle.stl"
+        />
+      </geometry>
+    </collision>
+    <inertial>
+      <origin rpy="0 0 0" xyz="-0.01926824 5.001e-05 0.02222178" />
+      <mass value="2.969376448e-02" />
+      <inertia
+        ixx="9.42456e-06"
+        ixy="0.0"
+        ixz="3.9636e-06"
+        iyy="8.69056e-06"
+        iyz="0.0"
+        izz="8.33824e-06"
+      />
+    </inertial>
+  </link>
+  <link name="robotiq_85_left_finger_tip_link">
+    <visual>
+      <geometry>
+        <mesh
+          filename="package://robotiq_description/meshes/visual/2f_85/left_finger_tip.dae"
+        />
+      </geometry>
+    </visual>
+    <collision>
+      <geometry>
+        <mesh
+          filename="package://robotiq_description/meshes/collision/2f_85/left_finger_tip.stl"
+        />
+      </geometry>
+      <surface>
+        <friction>
+          <ode>
+            <mu1>100000.0</mu1>
+            <mu2>100000.0</mu2>
+          </ode>
+        </friction>
+        <contact>
+          <ode>
+            <kp>1e+5</kp>
+            <kd>1</kd>
+            <soft_cfm>0</soft_cfm>
+            <soft_erp>0.2</soft_erp>
+            <minDepth>0.002</minDepth>
+            <maxVel>0</maxVel>
+          </ode>
+        </contact>
+      </surface>
+    </collision>
+    <inertial>
+      <origin rpy="0 0 0" xyz="-0.01456706 -0.0008 0.01649701" />
+      <mass value="4.268588744e-02" />
+      <inertia
+        ixx="1.048152e-05"
+        ixy="0.0"
+        ixz="3.5232e-6"
+        iyy="1.197888e-05"
+        iyz="0.0"
+        izz="4.22784e-06"
+      />
+    </inertial>
+  </link>
+  <link name="robotiq_85_right_finger_tip_link">
+    <visual>
+      <geometry>
+        <mesh
+          filename="package://robotiq_description/meshes/visual/2f_85/right_finger_tip.dae"
+        />
+      </geometry>
+    </visual>
+    <collision>
+      <geometry>
+        <mesh
+          filename="package://robotiq_description/meshes/collision/2f_85/right_finger_tip.stl"
+        />
+      </geometry>
+      <surface>
+        <friction>
+          <ode>
+            <mu1>100000.0</mu1>
+            <mu2>100000.0</mu2>
+          </ode>
+        </friction>
+        <contact>
+          <ode>
+            <kp>1e+5</kp>
+            <kd>1</kd>
+            <soft_cfm>0</soft_cfm>
+            <soft_erp>0.2</soft_erp>
+            <minDepth>0.002</minDepth>
+            <maxVel>0</maxVel>
+          </ode>
+        </contact>
+      </surface>
+    </collision>
+    <inertial>
+      <origin rpy="0 0 0" xyz="0.01456706 5e-05 0.01649701" />
+      <mass value="4.268588744e-02" />
+      <inertia
+        ixx="1.048152e-05"
+        ixy="0.0"
+        ixz="-3.5232e-06"
+        iyy="1.197888e-05"
+        iyz="0.0"
+        izz="4.22784e-06"
+      />
+    </inertial>
+  </link>
+  <joint name="robotiq_85_base_joint" type="fixed">
+    <parent link="gripper_mount_link" />
+    <child link="robotiq_85_base_link" />
+    <origin rpy="0 0 0" xyz="0 0 0" />
+  </joint>
+  <joint name="robotiq_85_left_knuckle_joint" type="revolute">
+    <parent link="robotiq_85_base_link" />
+    <child link="robotiq_85_left_knuckle_link" />
+    <axis xyz="0 -1 0" />
+    <origin rpy="0 0 0" xyz="0.03060114 0.0 0.05490452" />
+    <limit effort="20" lower="0.0" upper="0.8" velocity="0.5" />
+  </joint>
+  <joint name="robotiq_85_right_knuckle_joint" type="revolute">
+    <parent link="robotiq_85_base_link" />
+    <child link="robotiq_85_right_knuckle_link" />
+    <axis xyz="0 1 0" />
+    <origin rpy="0 0 0" xyz="-0.03060114 0.0 0.05490452" />
+    <limit effort="20" lower="0.0" upper="0.8" velocity="0.5" />
+    <mimic joint="robotiq_85_left_knuckle_joint" multiplier="1" />
+  </joint>
+  <joint name="robotiq_85_left_finger_joint" type="fixed">
+    <parent link="robotiq_85_left_knuckle_link" />
+    <child link="robotiq_85_left_finger_link" />
+    <axis xyz="0 -1 0" />
+    <origin rpy="0 0 0" xyz="0.03152616 0.0 -0.00376347" />
+  </joint>
+  <joint name="robotiq_85_right_finger_joint" type="fixed">
+    <parent link="robotiq_85_right_knuckle_link" />
+    <child link="robotiq_85_right_finger_link" />
+    <axis xyz="0 1 0" />
+    <origin rpy="0 0 0" xyz="-0.03152616 0.0 -0.00376347" />
+  </joint>
+  <joint name="robotiq_85_left_inner_knuckle_joint" type="continuous">
+    <parent link="robotiq_85_base_link" />
+    <child link="robotiq_85_left_inner_knuckle_link" />
+    <axis xyz="0 -1 0" />
+    <origin rpy="0 0 0" xyz="0.0127 0.0 0.06142" />
+    <mimic joint="robotiq_85_left_knuckle_joint" multiplier="1" />
+  </joint>
+  <joint name="robotiq_85_right_inner_knuckle_joint" type="continuous">
+    <parent link="robotiq_85_base_link" />
+    <child link="robotiq_85_right_inner_knuckle_link" />
+    <axis xyz="0 1 0" />
+    <origin rpy="0 0 0" xyz="-0.0127 0.0 0.06142" />
+    <mimic joint="robotiq_85_left_knuckle_joint" multiplier="1" />
+  </joint>
+  <joint name="robotiq_85_left_finger_tip_joint" type="continuous">
+    <parent link="robotiq_85_left_finger_link" />
+    <child link="robotiq_85_left_finger_tip_link" />
+    <axis xyz="0 -1 0" />
+    <origin rpy="0 0 0" xyz="0.00563134 0.0 0.04718515" />
+    <mimic joint="robotiq_85_left_knuckle_joint" multiplier="-1" />
+  </joint>
+  <joint name="robotiq_85_right_finger_tip_joint" type="continuous">
+    <parent link="robotiq_85_right_finger_link" />
+    <child link="robotiq_85_right_finger_tip_link" />
+    <axis xyz="0 1 0" />
+    <origin rpy="0 0 0" xyz="-0.00563134 0.0 0.04718515" />
+    <mimic joint="robotiq_85_left_knuckle_joint" multiplier="-1" />
+  </joint>
   <!-- This link aligns the axes of the grasp frame to our required convention for motion planning tasks. -->
   <link name="grasp_link" />
